File: schematic/anemometre.kicad_pcb (KiCad board)
At the start: 2 copper layers, 69.2 x 72.4 mm, 38 parts, among them J1 Anemometre, J10 PWR_SEL, J2 AVR-ISP-6, J3 PORT_C_ADC, J4 PORT_B, J5 Opto_PB0, J6 TTL Serial, J7 INTs/Ts, J8 USB_B_Mini, J9 +5VDC, SW1 Reset, U1 ATmega328P-P, U2 4N25, U3 FT232RL, Y1 8MHz

Commit message: latest modifications and add raincounter sensor
Routing:
- net /MISO: track 61.9 -> 61.2 mm
Changed lines of the file:
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@@
-	)
-	(segment
-		(start 105.155 56.77)
-		(end 104.648 57.277)
-		(width 0.2)
-		(layer "F.Cu")
-		(net 12)
 	)
 	(segment

Commit message: Schematic and PCB upgraded to support temperature and rain sensors
Parts:
- added C9: 100nF, Capacitor_THT:C_Disc_D7.0mm_W2.5mm_P5.00mm, F.Cu at (131.5, 65.5)
- added J11: Rain_PB1, Connector_PinHeader_2.54mm:PinHeader_1x03_P2.54mm_Vertical, F.Cu at (131.5, 50.0)
- added J12: Temp/Rain, TerminalBlock_Phoenix:TerminalBlock_Phoenix_MKDS-1,5-4-5.08_1x04_P5.08mm_Horizontal, F.Cu at (147.5, 67.6)
- added J13: Temp_PB2, Connector_PinHeader_2.54mm:PinHeader_1x03_P2.54mm_Vertical, F.Cu at (125.5, 50.0)
- added R10: 220, Resistor_THT:R_Axial_DIN0204_L3.6mm_D1.6mm_P7.62mm_Horizontal, F.Cu at (137.0, 55.0)
- added R11: 4.7K, Resistor_THT:R_Axial_DIN0204_L3.6mm_D1.6mm_P7.62mm_Horizontal, F.Cu at (139.5, 67.6)
- added R9: 4.7K, Resistor_THT:R_Axial_DIN0204_L3.6mm_D1.6mm_P7.62mm_Horizontal, F.Cu at (134.5, 67.8)
- D5: value LED -> PWR_LED
- J1: value Anemometre -> Anemometer
- J2: value AVR-ISP-6 -> AVR-ISP
- J5: value Opto_PB0 -> Anemo_PB0
- moved J4 43.2 mm to (125.5, 26.0), turned to -90 degrees
- moved R1 17.9 mm to (127.4, 44.5)
- moved J5 16.4 mm to (125.5, 36.5), turned to 0 degrees
- moved R2 14.8 mm to (140.0, 24.5)
- moved J1 13.9 mm to (147.5, 42.7)
- moved J9 13.1 mm to (151.0, 84.5)
- moved D3 13.1 mm to (137.3, 87.0)
- moved D5 13.0 mm to (151.5, 77.0)
- moved U2 9.00 mm to (128.9, 36.5), turned to 0 degrees
- moved SW1 8.59 mm to (133.0, 75.5)
- moved C3 0.26 mm to (114.0, 49.7)
- moved C4 0.17 mm to (109.0, 56.0)
Connections:
- J4 pad 2: Net-(J4-Pin_2) -> Net-(J11-Pin_1)
- J4 pad 3: Net-(J4-Pin_3) -> Net-(J13-Pin_1)
- U1 pad 15: Net-(J4-Pin_2) -> Net-(J11-Pin_2)
- U1 pad 16: Net-(J4-Pin_3) -> Net-(J13-Pin_2)
Routing:
- net Net-(J11-Pin_2): track 0.00 -> 36.7 mm
- net Net-(J4-Pin_1): track 46.4 -> 10.5 mm, vias 1 -> 0
- net Net-(J4-Pin_2): track 33.2 -> 0.00 mm
- net Net-(J4-Pin_3): track 33.2 -> 0.00 mm
- net Net-(J12-Pin_3): track 0.00 -> 31.5 mm
- net Net-(J11-Pin_1): track 0.00 -> 31.3 mm
- net Net-(J13-Pin_2): track 0.00 -> 29.1 mm
- net +5V: track 194.9 -> 223.9 mm
- net Net-(J13-Pin_1): track 0.00 -> 27.9 mm
- net Net-(J5-Pin_2): track 34.8 -> 49.8 mm, vias 0 -> 1
- net /MOSI: track 61.0 -> 75.0 mm, vias 0 -> 1
- net Net-(J11-Pin_3): track 0.00 -> 14.0 mm
- net Net-(D5-A): track 18.1 -> 30.1 mm
- net Net-(D3-K): track 70.8 -> 82.1 mm
- net Net-(J12-Pin_2): track 0.00 -> 10.5 mm
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Other:
- board size 69.2 x 72.4 mm -> 84.4 x 72.4 mm
- board text added: "*PB0"
- board text added: "*PB1"
- board text added: "*PB2"
- board text added: "+5VDC"
- board text added: "Anemo"
- board text added: "Rain"
- board text added: "Temp"
- board text added: "WEATHER STATION 1.0"
- board text removed: "PB0"
- board text removed: "PB1"
- board text removed: "PB2"
- board text removed: "SIGNAL"

Commit message: Latest shcematic of IOExtesion board and latest Gerbers
Parts:
- moved SW1 7.50 mm to (140.5, 75.5)
- moved D5 1.50 mm to (153.0, 77.0)
- moved J1 1.50 mm to (149.0, 42.7)
- moved J12 1.50 mm to (149.0, 67.6)
- moved J9 1.50 mm to (152.5, 84.5)
Routing:
- net /RESET: track 112.1 -> 120.6 mm
- net Net-(J12-Pin_3): track 31.5 -> 33.0 mm
- net Net-(J12-Pin_2): track 10.5 -> 12.0 mm
- net Net-(J1-Pin_2): track 21.8 -> 23.3 mm
- net Net-(D5-A): track 30.1 -> 31.6 mm
- net Net-(D3-A): track 3.56 -> 5.06 mm
- net +24V: track 8.72 -> 10.2 mm
- net +5V: track 223.9 -> 224.6 mm
Other:
- board size 84.4 x 72.4 mm -> 84.5 x 72.4 mm
